File: Hackpad.kicad_sch (KiCad schematic)
At the start: 21 parts, among them SW1 SW_Push, SW10 RotaryEncoder_Switch, SW2 SW_Push, SW3 SW_Push, SW4 SW_Push, SW5 SW_Push, SW6 SW_Push, SW7 SW_Push, SW8 SW_Push, SW9 SW_Push, U1 MOUDLE-SEEEDUINO-XIAO, U2 ER_OLEDM0.91_1x-I2C

Commit message: ain
Connections:
- net OLED renamed R3
- net R3: no longer U1.5 (PA8_A4_D4_SDA), U1.6 (PA9_A5_D5_SCL), U2.3 (SCL), U2.4 (SDA)
- new net: U1.6 (PA9_A5_D5_SCL), U2.3 (SCL)
- new net OLED_SDA: U1.5 (PA8_A4_D4_SDA), U2.4 (SDA)
Changed lines of the file:
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@@
+	)
+	(junction
+		(at 189.23 92.71)
+		(diameter 0)
+		(color 0 0 0 0)
 	)
 	(junction
@@
 	(wire
 		(pts
-			(xy 127 133.35) (xy 187.96 133.35)
+			(xy 127 133.35) (xy 185.42 133.35)
 		)
 		(stroke
@@
 	(wire
 		(pts
+			(xy 123.19 116.84) (xy 123.19 133.35)
+		)
+		(stroke
+			(width 0)
+			(type default)
+		)
+	)
+	(wire
+		(pts
 			(xy 160.02 93.98) (xy 119.38 93.98)
 		)
@@
 	(wire
 		(pts
+			(xy 119.38 124.46) (xy 127 124.46)
+		)
+		(stroke
+			(width 0)
+			(type default)
+		)
+	)
+	(wire
+		(pts
 			(xy 101.6 144.78) (xy 104.14 144.78)
 		)
@@
 	(wire
 		(pts
-			(xy 123.19 116.84) (xy 123.19 133.35)
-		)
-		(stroke
-			(width 0)
-			(type default)
-		)
-	)
-	(wire
-		(pts
 			(xy 189.23 95.25) (xy 189.23 127)
 		)
@@
 	(wire
 		(pts
+			(xy 120.65 121.92) (xy 127 121.92)
+		)
+		(stroke
+			(width 0)
+			(type default)
+		)
+	)
+	(wire
+		(pts
 			(xy 101.6 101.6) (xy 104.14 101.6)
 		)
@@
 	(wire
 		(pts
-			(xy 119.38 124.46) (xy 127 124.46)
-		)
-		(stroke
-			(width 0)
-			(type default)
-		)
-	)
-	(wire
-		(pts
 			(xy 66.04 114.3) (xy 91.44 114.3)
 		)
@@
 	(wire
 		(pts
-			(xy 120.65 121.92) (xy 127 121.92)
-		)
-		(stroke
-			(width 0)
-			(type default)
-		)
-	)
-	(wire
-		(pts
 			(xy 86.36 132.08) (xy 172.72 132.08)
 		)
@@
 	(wire
 		(pts
-			(xy 187.96 90.17) (xy 189.23 90.17)
+			(xy 185.42 90.17) (xy 189.23 90.17)
 		)
 		(stroke
@@
 	(wire
 		(pts
-			(xy 187.96 133.35) (xy 187.96 90.17)
+			(xy 185.42 133.35) (xy 185.42 90.17)
 		)
 		(stroke
@@
 		)
 	)
-	(label "OLED"
-		(at 123.19 124.46 0)
+	(label "OLED_SDA"
+		(at 124.46 121.92 0)
 		(effects
 			(font
-				(size 1.27 1.27)
-			)
-			(justify left bottom)
-		)
-	)
-	(label "OLED"
-		(at 123.19 121.92 0)
-		(effects
-			(font
